File: reembox_board/rev1/reembox.brd (EAGLE design)
At the start: 100 x 80 mm, 71 parts, among them IC1 MEGA32-P, IC10 LM3940, IC11 RFM12, IC2 ENC28J60-DIL, IC3 PCF8574P, IC4 PCA9685PW, IC5 ULN2803, IC6 ULN2803, IC7 MAX485, IC8 RFM12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

Commit message: pantries updated + ethersex pinning file
Parts:
- C10, C12: value 10uF -> NC
- C14: value 10uF -> 0,47uF
- IC1: value MEGA32-P -> MEGA644P
- IC9: value LM3940 -> RECOM R-78E5.0-0.5
- R15: value 33 -> NC
- R18: value 220 -> 2,2k
- R20: value 1k -> 1,2k
- R3, R4, R5, R6: value 50 -> 47
Changed lines of the file:
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@@
 </autorouter>
 <elements>
-<element name="IC1" library="atmel" package="DIL40" value="MEGA32-P" x="41.91" y="43.815">
+<element name="IC1" library="atmel" package="DIL40" value="MEGA644P" x="41.91" y="43.815">
 <attribute name="OC_NEWARK" value="51P1794" x="104.14" y="33.655" size="1.778" layer="27" display="off"/>
 <attribute name="MPN" value="ATMEGA32-16PU" x="104.14" y="33.655" size="1.778" layer="27" display="off"/>
@@
 <attribute name="VALUE" x="8.255" y="73.025" size="1.27" layer="27" ratio="10"/>
 </element>
-<element name="R15" library="rcl" package="0207/10" value="33" x="3.81" y="65.7225" smashed="yes" rot="R270">
+<element name="R15" library="rcl" package="0207/10" value="NC" x="3.81" y="65.7225" smashed="yes" rot="R270">
 <attribute name="NAME" x="3.1115" y="67.818" size="1.27" layer="25" ratio="10" rot="R270"/>
 <attribute name="VALUE" x="3.175" y="67.9831" size="1.27" layer="27" ratio="10" rot="R270"/>
@@
 <attribute name="VALUE" x="56.7944" y="25.4" size="1.27" layer="27" ratio="10"/>
 </element>
-<element name="R20" library="NetIO" package="RCL_0207/2V" value="1k" x="48.26" y="58.7375" smashed="yes">
+<element name="R20" library="NetIO" package="RCL_0207/2V" value="1,2k" x="48.26" y="58.7375" smashed="yes">
 <attribute name="NAME" x="51.689" y="57.7215" size="1.27" layer="25" ratio="10" rot="R90"/>
 <attribute name="VALUE" x="48.514" y="56.5277" size="1.27" layer="27" ratio="10"/>
@@
 <attribute name="VALUE" x="22.225" y="33.655" size="1.778" layer="27" ratio="10"/>
 </element>
-<element name="R5" library="rcl" package="0207/2V" value="50" x="25.4" y="20.6375" smashed="yes" rot="R90">
+<element name="R5" library="rcl" package="0207/2V" value="47" x="25.4" y="20.6375" smashed="yes" rot="R90">
 <attribute name="NAME" x="24.384" y="20.5867" size="1.27" layer="25" ratio="10" rot="R90"/>
 <attribute name="VALUE" x="27.6352" y="20.5867" size="1.27" layer="27" ratio="10" rot="R90"/>
 </element>
-<element name="R3" library="rcl" package="0207/2V" value="50" x="21.2725" y="8.255" smashed="yes" rot="R90">
+<element name="R3" library="rcl" package="0207/2V" value="47" x="21.2725" y="8.255" smashed="yes" rot="R90">
 <attribute name="NAME" x="20.2565" y="8.2042" size="1.27" layer="25" ratio="10" rot="R90"/>
 <attribute name="VALUE" x="23.5077" y="8.2042" size="1.27" layer="27" ratio="10" rot="R90"/>
 </element>
-<element name="R4" library="rcl" package="0207/2V" value="50" x="25.4" y="8.255" smashed="yes" rot="R90">
+<element name="R4" library="rcl" package="0207/2V" value="47" x="25.4" y="8.255" smashed="yes" rot="R90">
 <attribute name="NAME" x="24.384" y="8.2042" size="1.27" layer="25" ratio="10" rot="R90"/>
 <attribute name="VALUE" x="27.6352" y="8.2042" size="1.27" layer="27" ratio="10" rot="R90"/>
 </element>
-<element name="R6" library="rcl" package="0207/2V" value="50" x="21.2725" y="20.6375" smashed="yes" rot="R90">
+<element name="R6" library="rcl" package="0207/2V" value="47" x="21.2725" y="20.6375" smashed="yes" rot="R90">
 <attribute name="NAME" x="20.2565" y="20.5867" size="1.27" layer="25" ratio="10" rot="R90"/>
 <attribute name="VALUE" x="23.5077" y="20.5867" size="1.27" layer="27" ratio="10" rot="R90"/>
@@
 <attribute name="VALUE" x="7.8486" y="65.405" size="1.27" layer="27" ratio="10" rot="R270"/>
 </element>
-<element name="IC9" library="v-reg" package="78XXS" value="LM3940" x="97.155" y="46.6725" smashed="yes" rot="R270">
+<element name="IC9" library="v-reg" package="78XXS" value="RECOM R-78E5.0-0.5" x="97.155" y="46.6725" smashed="yes" rot="R270">
 <attribute name="NAME" x="97.4598" y="47.9425" size="1.27" layer="25" ratio="10" rot="R270"/>
 <attribute name="VALUE" x="89.535" y="51.7525" size="1.27" layer="27" ratio="10" rot="R270"/>
 </element>
-<element name="C14" library="rcl" package="E2,5-6" value="10uF" x="85.4075" y="49.53" smashed="yes" rot="R270">
+<element name="C14" library="rcl" package="E2,5-6" value="0,47uF" x="85.4075" y="49.53" smashed="yes" rot="R270">
 <attribute name="NAME" x="88.519" y="44.0055" size="1.27" layer="25" ratio="10" rot="R270"/>
 <attribute name="VALUE" x="82.7405" y="46.863" size="1.27" layer="27" ratio="10" rot="R270"/>
 </element>
-<element name="C10" library="rcl" package="E2,5-6" value="10uF" x="78.74" y="43.4975" smashed="yes" rot="R90">
+<element name="C10" library="rcl" package="E2,5-6" value="NC" x="78.74" y="43.4975" smashed="yes" rot="R90">
 <attribute name="NAME" x="81.788" y="48.006" size="1.27" layer="25" ratio="10" rot="R180"/>
 <attribute name="VALUE" x="81.407" y="46.1645" size="1.27" layer="27" ratio="10" rot="R90"/>
@@
 <attribute name="VALUE" x="88.0745" y="38.862" size="1.27" layer="27" ratio="10" rot="R90"/>
 </element>
-<element name="C12" library="rcl" package="E2,5-6" value="10uF" x="85.4075" y="42.8625" smashed="yes" rot="R90">
+<element name="C12" library="rcl" package="E2,5-6" value="NC" x="85.4075" y="42.8625" smashed="yes" rot="R90">
 <attribute name="NAME" x="89.5985" y="48.0695" size="1.27" layer="25" ratio="10" rot="R90"/>
 <attribute name="VALUE" x="88.0745" y="45.5295" size="1.27" layer="27" ratio="10" rot="R90"/>
@@
 <attribute name="VALUE" x="82.55" y="34.925" size="1.016" layer="27" ratio="10" rot="R90"/>
 </element>
-<element name="R18" library="rcl" package="0207/2V" value="220" x="73.3425" y="44.7675"/>
+<element name="R18" library="rcl" package="0207/2V" value="2,2k" x="73.3425" y="44.7675"/>
 <element name="IR2" library="con-molex" package="22-23-2021" value="IR" x="41.5925" y="62.865" smashed="yes" rot="R180">
 <attribute name="OC_NEWARK" value="25C3832" x="41.5925" y="62.865" size="1.778" layer="27" rot="R180" display="off"/>
